File: RC_Charger_MainBoard/30Vboost.kicad_sch (KiCad schematic)
At the start: 13 parts, among them U4 LM5001MA

Commit message: Change components for costdown
Parts:
- C3: value 100n -> 0.1u
- C5: footprint Capacitor_SMD:CP_Elec_10x10 -> Capacitor_SMD:CP_Elec_4x5.7
- L1: footprint Inductor_SMD:L_Bourns-SRU1028_10.0x10.0mm -> Inductor_SMD:L_Taiyo-Yuden_NR-80xx_HandSoldering
Changed lines of the file:
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@@
       (effects (font (size 1.27 1.27)) (justify left))
     )
-    (property "Footprint" "Capacitor_SMD:CP_Elec_10x10" (at 150.8252 77.47 0)
+    (property "Footprint" "Capacitor_SMD:CP_Elec_4x5.7" (at 150.8252 77.47 0)
       (effects (font (size 1.27 1.27)) hide)
     )
@@
       (effects (font (size 1.27 1.27)))
     )
-    (property "Footprint" "Inductor_SMD:L_Bourns-SRU1028_10.0x10.0mm" (at 132.08 69.85 0)
+    (property "Footprint" "Inductor_SMD:L_Taiyo-Yuden_NR-80xx_HandSoldering" (at 132.08 69.85 0)
       (effects (font (size 1.27 1.27)) hide)
     )
@@
       (effects (font (size 1.27 1.27)) (justify left))
     )
-    (property "Value" "100n" (at 95.25 74.93 0)
-      (effects (font (size 1.27 1.27)) (justify left))
-    )
+    (property "Value" "0.1u" (at 95.25 74.93 0)
+      (effects (font (size 1.27 1.27)) (justify left))
+    )
