File: RC_Charger_MainBoard/RC_Charger_MainBoard.kicad_sch (KiCad schematic)
At the start: 25 parts, among them J24 Conn_02x03_Odd_Even, J9 Conn_02x03_Odd_Even, U55 NUCLEO-H745ZI-Q, U56 L7805

Commit message: Change components for costdown
Parts:
- removed C25: 10p, Capacitor_SMD:C_0603_1608Metric, symbol Device:C
- removed C25: 4.7u, Capacitor_SMD:C_0603_1608Metric, symbol Device:C
- removed C25: 47p, Capacitor_SMD:C_0603_1608Metric, symbol Device:C
- removed C25: 12n, Capacitor_SMD:C_0603_1608Metric, symbol Device:C
- removed R7: 16.9k, Resistor_SMD:R_0603_1608Metric, symbol Device:R
- removed R7: 12.1k, Resistor_SMD:R_0603_1608Metric, symbol Device:R
- R6: value 36.5k -> 10k
- R6: value 53.6k -> 10k
- R7: value 10.2k -> 3.24k
- R7: value 11.7k -> 5.9k
Other:
- sheet 3V3 Buck ports: added none; removed COMP
- sheet 5V Buck ports: added none; removed COMP
