File: RC_Charger/IOMCU.kicad_sch (KiCad schematic)
At the start: 22 parts, among them J2 SWD, SW2 SW_DIP_x03, U15 STM32F103C8Tx, Y1 8M

Commit message: Add full bom and final pcb design
Parts:
- R58, R59: value 68 -> 100
Changed lines of the file:
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@@
       (effects (font (size 1.27 1.27)) (justify left))
     )
-    (property "Value" "68" (at 41.91 85.09 0)
+    (property "Value" "100" (at 41.91 85.09 0)
       (effects (font (size 1.27 1.27)) (justify left))
     )
@@
       (effects (font (size 1.27 1.27)) (justify left))
     )
-    (property "Value" "68" (at 30.48 85.09 0)
-      (effects (font (size 1.27 1.27)) (justify left))
-    )
+    (property "Value" "100" (at 30.48 85.09 0)
+      (effects (font (size 1.27 1.27)) (justify left))
+    )
