File: RC_Charger/battstage.kicad_sch (KiCad schematic)
At the start: 8 parts, among them J11 PWR1_DBG, J16 BAT, K5 Relay_SPST-NO, Q22 AO3400A, U59 INA240A1D

Commit message: Add full bom and final pcb design
Parts:
- removed K5: Relay_SPST-NO, Samacsys:T9GV5L145, symbol Relay:Relay_SPST-NO
- added K1: G2RL-1A-E, Relay_THT:Relay_SPST_Omron_G2RL-1A-E, symbol Relay:G2RL-1A-E
Connections:
- net +5V: now also K1.A1
- net IOMCU/VOUT: now also K1.13
- net at J16.2 (Pin_2), R249.1, U59.8 (+): now also K1.14
- net at D5.2 (A), Q22.3 (D): now also K1.A2
Changed lines of the file:
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@@
   (junction (at 76.2 121.92) (diameter 0) (color 0 0 0 0)
   )
-  (junction (at 88.9 91.44) (diameter 0) (color 0 0 0 0)
-  )
   (junction (at 97.79 64.77) (diameter 0) (color 0 0 0 0)
   )
+  (junction (at 123.19 92.71) (diameter 0) (color 0 0 0 0)
+  )
   (junction (at 60.96 121.92) (diameter 0) (color 0 0 0 0)
   )
@@
     (stroke (width 0) (type default))
   )
-  (wire (pts (xy 123.19 91.44) (xy 123.19 95.25))
+  (wire (pts (xy 107.95 91.44) (xy 88.9 91.44))
+    (stroke (width 0) (type default))
+  )
+  (wire (pts (xy 123.19 91.44) (xy 123.19 92.71))
     (stroke (width 0) (type default))
   )
@@
     (stroke (width 0) (type default))
   )
+  (wire (pts (xy 88.9 106.68) (xy 110.49 106.68))
+    (stroke (width 0) (type default))
+  )
   (wire (pts (xy 100.33 123.19) (xy 100.33 121.92))
     (stroke (width 0) (type default))
@@
     (stroke (width 0) (type default))
   )
+  (wire (pts (xy 107.95 102.87) (xy 107.95 91.44))
+    (stroke (width 0) (type default))
+  )
   (wire (pts (xy 106.68 133.35) (xy 107.95 133.35))
     (stroke (width 0) (type default))
@@
     (stroke (width 0) (type default))
   )
-  (wire (pts (xy 107.95 102.87) (xy 107.95 109.22))
-    (stroke (width 0) (type default))
-  )
   (wire (pts (xy 78.74 64.77) (xy 97.79 64.77))
     (stroke (width 0) (type default))
@@
     (stroke (width 0) (type default))
   )
-  (wire (pts (xy 107.95 109.22) (xy 88.9 109.22))
-    (stroke (width 0) (type default))
-  )
   (wire (pts (xy 152.4 68.58) (xy 157.48 68.58))
     (stroke (width 0) (type default))
@@
     (stroke (width 0) (type default))
   )
+  (wire (pts (xy 123.19 92.71) (xy 123.19 95.25))
+    (stroke (width 0) (type default))
+  )
   (wire (pts (xy 152.4 81.28) (xy 153.67 81.28))
     (stroke (width 0) (type default))
@@
     (stroke (width 0) (type default))
   )
-  (wire (pts (xy 88.9 91.44) (xy 123.19 91.44))
-    (stroke (width 0) (type default))
-  )
   (wire (pts (xy 113.03 64.77) (xy 120.65 64.77))
     (stroke (width 0) (type default))
@@
     (stroke (width 0) (type default))
   )
+  (wire (pts (xy 110.49 92.71) (xy 123.19 92.71))
+    (stroke (width 0) (type default))
+  )
   (wire (pts (xy 115.57 125.73) (xy 156.21 125.73))
     (stroke (width 0) (type default))
@@
     (stroke (width 0) (type default))
   )
-  (wire (pts (xy 88.9 109.22) (xy 88.9 106.68))
+  (wire (pts (xy 110.49 106.68) (xy 110.49 92.71))
     (stroke (width 0) (type default))
   )
@@
   (hierarchical_label "SCL" (shape input) (at 96.52 77.47 180) (fields_autoplaced)
     (effects (font (size 1.27 1.27)) (justify right))
-  )
-  (symbol (lib_id "power:+5V") (at 88.9 91.44 0) (unit 1)
-    (in_bom yes) (on_board yes) (dnp no) (fields_autoplaced)
-    (property "Reference" "#PWR053" (at 88.9 95.25 0)
-      (effects (font (size 1.27 1.27)) hide)
-    )
-    (property "Value" "+5V" (at 88.9 86.36 0)
-      (effects (font (size 1.27 1.27)))
-    )
-    (property "Footprint" "" (at 88.9 91.44 0)
-      (effects (font (size 1.27 1.27)) hide)
-    )
-    (property "Datasheet" "" (at 88.9 91.44 0)
-      (effects (font (size 1.27 1.27)) hide)
-    )
-    (pin "1")
-    (instances
-      (project "RC_Charger"
-        (path "/0902a6fd-0525-43c9-a70c-b987859163f6"
-          (reference "#PWR053") (unit 1)
-        )
-        (path "/0902a6fd-0525-43c9-a70c-b987859163f6/44385ac6-2dac-4298-a0ef-bab3c9dededd"
-          (reference "#PWR054") (unit 1)
-        )
-        (path "/0902a6fd-0525-43c9-a70c-b987859163f6/1ee38852-1559-48b6-8a70-6102d2608532"
-          (reference "#PWR055") (unit 1)
-        )
-      )
-      (project "RC_Charger_MainBoard"
-        (path "/43d535c7-5e30-4b88-a9b0-e712620238f3"
-          (reference "#PWR017") (unit 1)
-        )
-      )
-    )
   )
   (symbol (lib_id "Amplifier_Current:INA240A1D") (at 107.95 125.73 0) (unit 1)
@@
     )
   )
-  (symbol (lib_id "Relay:Relay_SPST-NO") (at 83.82 99.06 180) (unit 1)
-    (in_bom yes) (on_board yes) (dnp no) (fields_autoplaced)
-    (property "Reference" "K5" (at 95.25 97.79 0)
+  (symbol (lib_id "Relay:G2RL-1A-E") (at 83.82 99.06 180) (unit 1)
+    (in_bom yes) (on_board yes) (dnp no) (fields_autoplaced)
+    (property "Reference" "K1" (at 95.25 97.79 0)
       (effects (font (size 1.27 1.27)) (justify right))
     )
-    (property "Value" "Relay_SPST-NO" (at 95.25 100.33 0)
+    (property "Value" "G2RL-1A-E" (at 95.25 100.33 0)
       (effects (font (size 1.27 1.27)) (justify right))
     )
-    (property "Footprint" "Samacsys:T9GV5L145" (at 72.39 97.79 0)
+    (property "Footprint" "Relay_THT:Relay_SPST_Omron_G2RL-1A-E" (at 72.39 97.79 0)
       (effects (font (size 1.27 1.27)) (justify left) hide)
     )
-    (property "Datasheet" "~" (at 83.82 99.06 0)
-      (effects (font (size 1.27 1.27)) hide)
-    )
+    (property "Datasheet" "https://omronfs.omron.com/en_US/ecb/products/pdf/en-g2rl.pdf" (at 83.82 99.06 0)
+      (effects (font (size 1.27 1.27)) hide)
+    )
+    (pin "A1")
     (pin "A2")
+    (pin "13")
     (pin "14")
-    (pin "13")
-    (pin "A1")
-    (instances
-      (project "RC_Charger"
-        (path "/0902a6fd-0525-43c9-a70c-b987859163f6/44385ac6-2dac-4298-a0ef-bab3c9dededd"
-          (reference "K5") (unit 1)
-        )
-        (path "/0902a6fd-0525-43c9-a70c-b987859163f6/1ee38852-1559-48b6-8a70-6102d2608532"
-          (reference "K6") (unit 1)
-        )
-      )
+    (instances
+      (project "RC_Charger"
+        (path "/0902a6fd-0525-43c9-a70c-b987859163f6/44385ac6-2dac-4298-a0ef-bab3c9dededd"
+          (reference "K1") (unit 1)
+        )
+        (path "/0902a6fd-0525-43c9-a70c-b987859163f6/1ee38852-1559-48b6-8a70-6102d2608532"
+          (reference "K2") (unit 1)
+        )
+      )
+    )
+  )
+  (symbol (lib_id "power:+5V") (at 123.19 91.44 0) (unit 1)
+    (in_bom yes) (on_board yes) (dnp no) (fields_autoplaced)
+    (property "Reference" "#PWR053" (at 123.19 95.25 0)
+      (effects (font (size 1.27 1.27)) hide)
+    )
+    (property "Value" "+5V" (at 123.19 86.36 0)
+      (effects (font (size 1.27 1.27)))
+    )
+    (property "Footprint" "" (at 123.19 91.44 0)
+      (effects (font (size 1.27 1.27)) hide)
+    )
+    (property "Datasheet" "" (at 123.19 91.44 0)
+      (effects (font (size 1.27 1.27)) hide)
+    )
+    (pin "1")
+    (instances
+      (project "RC_Charger"
+        (path "/0902a6fd-0525-43c9-a70c-b987859163f6"
+          (reference "#PWR053") (unit 1)
+        )
+        (path "/0902a6fd-0525-43c9-a70c-b987859163f6/44385ac6-2dac-4298-a0ef-bab3c9dededd"
+          (reference "#PWR054") (unit 1)
+        )
+        (path "/0902a6fd-0525-43c9-a70c-b987859163f6/1ee38852-1559-48b6-8a70-6102d2608532"
+          (reference "#PWR055") (unit 1)
+        )
+      )
+      (project "RC_Charger_MainBoard"
+        (path "/43d535c7-5e30-4b88-a9b0-e712620238f3"
+          (reference "#PWR017") (unit 1)
+        )
+      )
